File: IQModulator.brd (EAGLE design)
At the start: 141 x 88.9 mm, 182 parts, among them IC1 LP2992, IC2 TLV2464CDD, IC4 SN74CBTLV3253D, IC5 FT232RL-FULLSSOP, IC6 74AC74D, IC7 SI5351A_DEVICE_SMD, IC8 MEGA8-AI, Q1 16MHz, Q2 25MHz, X1 KLBR4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

Commit message: Layout done
Parts:
- moved U$9 14.8 mm to (48.3, 72.4), turned to 0 degrees
- moved T6 2.54 mm to (10.2, 32.4)
- moved D1 2.29 mm to (40.0, 79.4), turned to 180 degrees
- moved C30 1.80 mm to (9.53, 27.9), turned to 270 degrees
- moved C26 1.27 mm to (17.8, 40.0)
- moved T2 1.27 mm to (15.9, 62.9)
- moved C46 0.90 mm to (18.4, 3.81), turned to 270 degrees
- moved C25 0.64 mm to (16.5, 32.4)
- moved C27 0.64 mm to (21.6, 36.8), turned to 180 degrees
- moved L10 0.64 mm to (16.5, 37.5)
- moved L9 0.63 mm to (21.6, 33.0), turned to 180 degrees
Routing:
- net +5V: track 82.1 -> 361.7 mm, vias 0 -> 3
- net LOAD: track 9.04 -> 127.0 mm
- net CONTROL2: track 16.0 -> 121.8 mm, vias 1 -> 4
- net CONTROL6: track 31.9 -> 111.9 mm, vias 1 -> 4
- net CONTROL1: track 13.8 -> 93.1 mm, vias 1 -> 2
- net CONTROL3: track 12.1 -> 84.0 mm, vias 1 -> 4
- net PA_OUT: track 0.00 -> 67.8 mm, vias 0 -> 1
- net CONTROL8: track 35.5 -> 97.5 mm, vias 1 -> 2
- net CONTROL5: track 50.3 -> 107.6 mm, vias 1 -> 4
- net N$30: track 0.00 -> 48.4 mm, vias 0 -> 1
- net N$43: track 0.00 -> 48.4 mm
- net N$47: track 0.00 -> 42.7 mm
- net N$45: track 0.00 -> 41.2 mm, vias 0 -> 1
- net CONTROL7: track 32.4 -> 69.2 mm, vias 1 -> 2
- net N$38: track 0.00 -> 36.8 mm
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
Commit message: error handling
Parts:
- turned C5 to 270 degrees
Routing:
- net SCL: track 56.7 -> 92.7 mm, vias 2 -> 4
- net +5V: track 361.7 -> 370.6 mm
- net N$12: track 31.5 -> 29.6 mm
- net N$45: track 41.2 -> 42.6 mm, vias 1 -> 0
- net PA_OUT: track 67.8 -> 68.7 mm, vias 1 -> 0
- net N$46: track 40.7 -> 41.1 mm, vias 1 -> 0

Commit message: updated board
Routing:
- net +5V: track 370.6 -> 363.5 mm
- net SCL: track 92.7 -> 93.5 mm
- net GND: vias 7 -> 8
Other:
- board text added: "GND"
- board text added: "IQ-Modulator Bachelorarbeit Pirmin Schöder"
Changed lines of the file:
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@@
 <grid distance="25" unitdist="mil" unit="mil" style="lines" multiple="1" display="yes" altdistance="0.025" altunitdist="inch" altunit="inch"/>
 <layers>
-<layer number="1" name="Top" color="4" fill="1" visible="yes" active="yes"/>
+<layer number="1" name="Top" color="4" fill="1" visible="no" active="yes"/>
 <layer number="2" name="Route2" color="1" fill="3" visible="no" active="no"/>
 <layer number="3" name="Route3" color="4" fill="3" visible="no" active="no"/>
 <layer number="14" name="Route14" color="1" fill="6" visible="no" active="no"/>
 <layer number="15" name="Route15" color="4" fill="6" visible="no" active="no"/>
-<layer number="16" name="Bottom" color="1" fill="1" visible="yes" active="yes"/>
-<layer number="17" name="Pads" color="2" fill="1" visible="yes" active="yes"/>
-<layer number="18" name="Vias" color="2" fill="1" visible="yes" active="yes"/>
-<layer number="19" name="Unrouted" color="6" fill="1" visible="yes" active="yes"/>
+<layer number="16" name="Bottom" color="1" fill="1" visible="no" active="yes"/>
+<layer number="17" name="Pads" color="2" fill="1" visible="no" active="yes"/>
+<layer number="18" name="Vias" color="2" fill="1" visible="no" active="yes"/>
+<layer number="19" name="Unrouted" color="6" fill="1" visible="no" active="yes"/>
 <layer number="20" name="Dimension" color="15" fill="1" visible="yes" active="yes"/>
 <layer number="21" name="tPlace" color="7" fill="1" visible="yes" active="yes"/>
-<layer number="22" name="bPlace" color="7" fill="1" visible="yes" active="yes"/>
-<layer number="23" name="tOrigins" color="15" fill="1" visible="yes" active="yes"/>
-<layer number="24" name="bOrigins" color="15" fill="1" visible="yes" active="yes"/>
-<layer number="25" name="tNames" color="7" fill="1" visible="no" active="yes"/>
+<layer number="22" name="bPlace" color="7" fill="1" visible="no" active="yes"/>
+<layer number="23" name="tOrigins" color="15" fill="1" visible="no" active="yes"/>
+<layer number="24" name="bOrigins" color="15" fill="1" visible="no" active="yes"/>
+<layer number="25" name="tNames" color="7" fill="1" visible="yes" active="yes"/>
 <layer number="26" name="bNames" color="7" fill="1" visible="no" active="yes"/>
 <layer number="27" name="tValues" color="7" fill="1" visible="no" active="yes"/>
@@
 <wire x1="140.97" y1="88.9" x2="0" y2="88.9" width="0" layer="20"/>
 <wire x1="0" y1="88.9" x2="0" y2="0" width="0" layer="20"/>
+<text x="1.27" y="83.82" size="1.778" layer="22" font="vector">IQ-Modulator Bachelorarbeit
+             Pirmin Schöder</text>
+<text x="57.785" y="3.81" size="1.778" layer="21" font="vector">GND</text>
+<text x="76.835" y="3.81" size="1.778" layer="21" font="vector">GND</text>
 </plain>
 <attributes>
@@
 <param name="mtCopper" value="0.035mm 0.035mm 0.035mm 0.035mm 0.035mm 0.035mm 0.035mm 0.035mm 0.035mm 0.035mm 0.035mm 0.035mm 0.035mm 0.035mm 0.035mm 0.035mm"/>
 <param name="mtIsolate" value="1.5mm 0.15mm 0.2mm 0.15mm 0.2mm 0.15mm 0.2mm 0.15mm 0.2mm 0.15mm 0.2mm 0.15mm 0.2mm 0.15mm 0.2mm"/>
-<param name="mdWireWire" value="7mil"/>
-<param name="mdWirePad" value="7mil"/>
-<param name="mdWireVia" value="7mil"/>
-<param name="mdPadPad" value="7mil"/>
-<param name="mdPadVia" value="7mil"/>
-<param name="mdViaVia" value="7mil"/>
+<param name="mdWireWire" value="8mil"/>
+<param name="mdWirePad" value="8mil"/>
+<param name="mdWireVia" value="8mil"/>
+<param name="mdPadPad" value="8mil"/>
+<param name="mdPadVia" value="8mil"/>
+<param name="mdViaVia" value="8mil"/>
 <param name="mdSmdPad" value="0mil"/>
 <param name="mdSmdVia" value="0mil"/>
@@
 <via x="114.935" y="53.34" extent="1-16" drill="0.6"/>
 <via x="74.295" y="60.96" extent="1-16" drill="0.6"/>
+<via x="68.58" y="55.245" extent="1-16" drill="0.6"/>
 <wire x1="127" y1="34.61" x2="127" y2="36.51" width="0" layer="19" extent="1-1"/>
 <wire x1="97.155" y1="66.36" x2="100.645" y2="62.865" width="0" layer="19" extent="1-1"/>
@@
 <wire x1="20.64" y1="36.83" x2="20.64" y2="33.07" width="0.4064" layer="1"/>
 <wire x1="20.64" y1="33.07" x2="20.69" y2="33.02" width="0.4064" layer="1"/>
-<wire x1="17.46" y1="32.385" x2="17.46" y2="37.415" width="0.254" layer="1"/>
-<wire x1="17.46" y1="37.415" x2="17.41" y2="37.465" width="0.254" layer="1"/>
-<wire x1="17.46" y1="37.415" x2="20.055" y2="37.415" width="0.254" layer="1"/>
-<wire x1="20.055" y1="37.415" x2="20.64" y2="36.83" width="0.254" layer="1"/>
+<wire x1="17.46" y1="32.385" x2="17.46" y2="37.415" width="0.3048" layer="1"/>
+<wire x1="17.46" y1="37.415" x2="17.41" y2="37.465" width="0.3048" layer="1"/>
+<wire x1="17.46" y1="37.415" x2="20.055" y2="37.415" width="0.3048" layer="1"/>
+<wire x1="20.055" y1="37.415" x2="20.64" y2="36.83" width="0.3048" layer="1"/>
 </signal>
 <signal name="FIL5_OUT">
@@
 <wire x1="10.205" y1="10.795" x2="10.205" y2="11.475" width="0.4064" layer="16"/>
 <wire x1="10.205" y1="11.475" x2="12.065" y2="13.335" width="0.4064" layer="16"/>
-<wire x1="12.065" y1="13.335" x2="35.56" y2="13.335" width="0.4064" layer="16"/>
-<wire x1="35.56" y1="13.335" x2="38.735" y2="10.16" width="0.4064" layer="16"/>
-<wire x1="38.735" y1="10.16" x2="41.275" y2="10.16" width="0.4064" layer="16"/>
-<wire x1="41.275" y1="10.16" x2="41.275" y2="12.11" width="0.4064" layer="16"/>
+<wire x1="12.065" y1="13.335" x2="37.465" y2="13.335" width="0.4064" layer="16"/>
 <wire x1="12.71" y1="36.195" x2="12.7" y2="36.195" width="0.4064" layer="1"/>
 <wire x1="12.7" y1="36.195" x2="12.7" y2="38.1" width="0.4064" layer="1"/>
@@
 <contactref element="R16" pad="1"/>
 <contactref element="IC8" pad="28"/>
-<wire x1="62.365" y1="17.29" x2="62.365" y2="18.28" width="0.254" layer="1"/>
-<wire x1="62.365" y1="18.28" x2="61.595" y2="19.05" width="0.254" layer="1"/>
-<wire x1="61.595" y1="19.05" x2="60.96" y2="19.05" width="0.254" layer="1"/>
-<wire x1="60.96" y1="19.05" x2="60.325" y2="19.685" width="0.254" layer="1"/>
 <via x="110.49" y="8.255" extent="1-16" drill="0.6"/>
 <wire x1="110.49" y1="8.255" x2="104.14" y2="8.255" width="0.3048" layer="1"/>
@@
 <via x="55.88" y="15.875" extent="1-16" drill="0.6"/>
 <wire x1="55.88" y1="15.875" x2="55.88" y2="19.685" width="0.254" layer="1"/>
-<wire x1="55.88" y1="19.685" x2="60.325" y2="19.685" width="0.254" layer="1"/>
+<wire x1="55.88" y1="19.685" x2="62.23" y2="19.685" width="0.254" layer="1"/>
+<wire x1="62.365" y1="17.29" x2="62.365" y2="19.55" width="0.254" layer="1"/>
+<wire x1="62.365" y1="19.55" x2="62.23" y2="19.685" width="0.254" layer="1"/>
 </signal>
 <signal name="SDA">
@@
 <wire x1="97.79" y1="12.38" x2="99.06" y2="11.11" width="0.3048" layer="1"/>
 <wire x1="103.143" y1="23.8506" x2="103.143" y2="25.673" width="0.3048" layer="1"/>
-<wire x1="103.143" y1="25.673" x2="104.775" y2="27.305" width="0.3048" layer="1"/>
-<wire x1="104.775" y1="27.305" x2="105.41" y2="27.305" width="0.3048" layer="1"/>
-<wire x1="105.41" y1="27.305" x2="106.68" y2="28.575" width="0.3048" layer="1"/>
-<wire x1="106.68" y1="28.575" x2="106.68" y2="30.8" width="0.3048" layer="1"/>
 <wire x1="103.143" y1="23.8506" x2="103.143" y2="21.863" width="0.3048" layer="1"/>
 <wire x1="103.143" y1="21.863" x2="102.87" y2="21.59" width="0.3048" layer="1"/>
@@
 <wire x1="101.543" y1="18.358" x2="100.743" y2="17.558" width="0.3048" layer="1"/>
 <wire x1="100.743" y1="15.2654" x2="100.743" y2="17.558" width="0.3048" layer="1"/>
+<wire x1="103.143" y1="25.673" x2="106.68" y2="29.21" width="0.3048" layer="1"/>
+<wire x1="106.68" y1="29.21" x2="106.68" y2="30.8" width="0.3048" layer="1"/>
 </signal>
 <signal name="N$19">
@@
 <contactref element="IC7" pad="9"/>
 <contactref element="X2" pad="1"/>
-<wire x1="63.365" y1="13.19" x2="63.365" y2="10.93" width="0.254" layer="1"/>
-<wire x1="63.365" y1="10.93" x2="63.5" y2="10.795" width="0.254" layer="1"/>
-<wire x1="63.5" y1="10.795" x2="64.77" y2="10.795" width="0.254" layer="1"/>
-<wire x1="64.77" y1="10.795" x2="69.85" y2="5.715" width="0.254" layer="1"/>
+<wire x1="64.135" y1="11.43" x2="69.85" y2="5.715" width="0.254" layer="1"/>
 <wire x1="69.85" y1="5.715" x2="70.41" y2="5.08" width="0.254" layer="1"/>
+<wire x1="63.365" y1="13.19" x2="63.365" y2="11.565" width="0.254" layer="1"/>
+<wire x1="63.365" y1="11.565" x2="63.5" y2="11.43" width="0.254" layer="1"/>
+<wire x1="63.5" y1="11.43" x2="64.135" y2="11.43" width="0.254" layer="1"/>
 </signal>
 <signal name="N$41">
@@
 <wire x1="13.97" y1="40.005" x2="12.1666" y2="40.005" width="0.3048" layer="1"/>
 <wire x1="12.1666" y1="40.005" x2="11.811" y2="39.6494" width="0.3048" layer="1"/>
-<wire x1="78.105" y1="13.97" x2="78.74" y2="13.335" width="0.3048" layer="16"/>
-<wire x1="78.74" y1="13.335" x2="85.09" y2="13.335" width="0.3048" layer="16"/>
-<wire x1="78.105" y1="13.97" x2="50.8" y2="13.97" width="0.3048" layer="16"/>
 <wire x1="50.8" y1="13.97" x2="48.895" y2="15.875" width="0.3048" layer="16"/>
 <via x="48.895" y="15.875" extent="1-16" drill="0.6"/>
@@
 <wire x1="44.45" y1="22.86" x2="43.18" y2="24.13" width="0.3048" layer="1"/>
 <via x="43.18" y="24.13" extent="1-16" drill="0.6"/>
+<wire x1="50.8" y1="13.97" x2="55.88" y2="13.97" width="0.3048" layer="16"/>
+<wire x1="55.88" y1="13.97" x2="56.515" y2="13.335" width="0.3048" layer="16"/>
+<wire x1="56.515" y1="13.335" x2="85.09" y2="13.335" width="0.3048" layer="16"/>
 </signal>
 <signal name="CONTROL6">
@@
 </board>
 </drawing>
+<compatibility>
+<note version="6.3" minversion="6.2.2" severity="warning">
+Since Version 6.2.2 text objects can contain more than one line,
+which will not be processed correctly with this version.
+</note>
+</compatibility>
 </eagle>
