File: IQModulator_mod.brd (EAGLE design)
At the start: 140.6 x 95.4 mm, 183 parts, among them IC1 LP2992, IC2 TLV2464CDD, IC4 SN74CBTLV3253D, IC5 FT232RL-FULLSSOP, IC6 74AC74D, IC7 SI5351A_DEVICE_SMD, IC8 MEGA8-AI, Q1 16MHz, Q2 25MHz

Commit message: Ready for gerbhouse
Parts:
- D1, D2, D3, D4, D5, D6, D7, D8: device diode:DO214AA -> diode:SOD323R_INFINEON
- moved C70 8.64 mm to (74.0, 91.8), turned to 0 degrees
- moved C61 3.59 mm to (63.8, 75.9)
- moved D2 3.18 mm to (9.53, 74.3)
- moved D1 2.54 mm to (43.2, 81.9), turned to 90 degrees
- moved D6 1.90 mm to (8.89, 38.7), turned to 270 degrees
Routing:
- net +5V: track 355.9 -> 346.1 mm
- net CONTROL4: track 74.0 -> 67.4 mm, vias 3 -> 2
- net N$49: track 20.2 -> 23.9 mm
- net N$38: track 36.8 -> 33.4 mm
- net N$48: track 37.9 -> 39.6 mm
- net N$47: track 42.7 -> 41.2 mm
- net SDA: track 78.1 -> 79.5 mm
- net N$39: track 35.6 -> 36.9 mm
- net N$30: track 48.4 -> 47.4 mm
- net CONTROL5: vias 4 -> 2
- net CONTROL6: vias 4 -> 2
Other:
- board text added: "IQ-Modulator Bachelorarbeit"
- board text added: "Pirmin Schöder"
- board text removed: "IQ-Modulator Bachelorarbeit - Pirmin Schöder"
